File: kicad_ci_test.kicad_sch (KiCad schematic)
At the start: 4 parts, among them J1 Conn_01x02_Female, J2 Conn_01x02_Female

Commit message: Migrated to KiCad 7.0.11
Parts:
- removed J1, J2: Conn_01x02_Female, Connector_Molex:Molex_KK-254_AE-6410-02A_1x02_P2.54mm_Vertical, symbol Connector:Conn_01x02_Female
- added J1, J2: Conn_01x02_Socket, Connector_Molex:Molex_KK-254_AE-6410-02A_1x02_P2.54mm_Vertical, symbol Connector:Conn_01x02_Socket
Connections:
- net GND: now also J1.2 (Pin_2), J2.2 (Pin_2)
- net at C1.1, R1.1: now also J2.1 (Pin_1)
- net at R1.2: now also J1.1 (Pin_1)
