File: kicad_ci_test.kicad_sch (KiCad schematic)
At the start: 4 parts, among them J1 Conn_01x02_Socket, J2 Conn_01x02_Socket

Commit message: Also set R1 tolerance in the simple example
Parts:
- R1: Tolerance (none) -> 5%
Changed lines of the file:
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@@
+			)
+		)
+		(property "Tolerance" "5%"
+			(at 101.6 67.31 90)
+			(effects
+				(font
+					(size 1.27 1.27)
+				)
+				(hide yes)
 			)
 		)
