File: test_subdir/test_subdir.kicad_sch (KiCad schematic)
At the start: 12 parts, among them J1 Conn_01x08_Male, J2 Conn_01x08_Male, J3 Conn_01x08_Male, J4 USB_B, J5 Conn_01x08_Male, J6 Conn_01x06_Male, U1 FT2232H, Y1 12 MHz

Commit message: Migrated the sub-dir example to KiCad 7.0.11
Parts:
- J1, J2, J3, J5: symbol Connector:Conn_01x08_Male -> Connector:Conn_01x08_Pin
- J6: symbol Connector:Conn_01x06_Male -> Connector:Conn_01x06_Pin
