File: test_subdir/test_subdir.kicad_pcb (KiCad board)
At the start: 4 copper layers, 49.8 x 48.2 mm, 12 parts, among them J1 Conn_01x08_Male, J2 Conn_01x08_Male, J3 Conn_01x08_Male, J4 USB_B, J5 Conn_01x08_Male, J6 Conn_01x06_Male, U1 FT2232H, Y1 12 MHz

Commit message: [Fixed] Use of "12k 1%" which is currently discouraged
Parts:
- R2: value 12k 1% -> 12k
Changed lines of the file:
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@@
 			)
 		)
-		(property "Datasheet" " ~"
+		(property "Datasheet" ""
 			(at 0 0 180)
 			(layer "F.Fab")
@@
 			)
 		)
-		(property "Value" "12k 1%"
+		(property "Value" "12k"
 			(at 2.54 2.37 0)
 			(layer "F.Fab")
@@
 					(thickness 0.15)
 				)
+			)
+		)
+		(property "Tolerance" "1%"
+			(at 0 0 180)
+			(unlocked yes)
+			(layer "F.Fab")
+			(hide yes)
+			(effects
+				(font
+					(size 1 1)
+					(thickness 0.15)
+				)
